File: Electricity & Electronics/Schematics/Schematics.kicad_sch (KiCad schematic)
At the start: 5 parts

Commit message: Latest
Parts:
- removed R1, R2, Rx: R, symbol Device:R
- removed Rs: R_Variable, symbol Device:R_Variable
- added BT2: 5V, symbol Device:Battery_Cell
- added BT3: 15V, symbol Device:Battery_Cell
- added L1: L, symbol Device:L
- added R, R2 (x2): 10k, symbol Device:R
- added R1 (x2), R3 (x2): 20k, symbol Device:R
- added S: SW_SPST, symbol Switch:SW_SPST
- BT1: value Battery_Cell -> 15V
Connections:
- net at BT1.1 (+): now also R1.1
- net at BT1.2 (-): now also R2.2, R3.1
- new net: BT2.2 (-), R1.1, R3.1
- new net: R1.2, R2.1, R3.2 (x2)
- new net: BT3.1 (+), S.1 (A)
- new net: BT3.2 (-), L1.1
- new net: BT2.1 (+), R2.2
- new net: L1.2, R.1
- new net: R.2, S.2 (B)
Other:
- note removed: "V1"
- note removed: "Vx"
